File: babyGroot.brd (EAGLE design)
At the start: 62.5 x 50 mm, 45 parts, among them IC1 ATMEGA168-20P, IC2 ULN2003AN, IC3 7805TV

Commit message: Add files via upload
Parts:
- C1: value (none) -> .1uF
- C2, C3: value (none) -> 22pF
- C4: value (none) -> 4.7uF
- C5: value (none) -> 0.47uF
- Q1: value (none) -> 16MHz
- R1, R2: value (none) -> 4.7k
- R3: value (none) -> 15k
- R4, R5, R6, R7, R8, R9: value (none) -> 470
Changed lines of the file:
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@@
 <attribute name="VALUE" x="33.993" y="15.635" size="1.27" layer="27" ratio="10" rot="R180"/>
 </element>
-<element name="R9" library="adafruit" package="0204V" value="" x="59" y="24" smashed="yes">
+<element name="R9" library="adafruit" package="0204V" value="470" x="59" y="24" smashed="yes">
 <attribute name="NAME" x="55.2674" y="23.5754" size="0.8128" layer="25" ratio="12"/>
 <attribute name="VALUE" x="56.8664" y="21.6886" size="1.27" layer="27" ratio="12"/>
 </element>
-<element name="R8" library="adafruit" package="0204V" value="" x="36.5" y="29" smashed="yes" rot="R270">
+<element name="R8" library="adafruit" package="0204V" value="470" x="36.5" y="29" smashed="yes" rot="R270">
 <attribute name="NAME" x="37.5922" y="28" size="0.8128" layer="25" ratio="12"/>
 <attribute name="VALUE" x="34.1886" y="31.1336" size="1.27" layer="27" ratio="12" rot="R270"/>
 </element>
-<element name="R7" library="adafruit" package="0204V" value="" x="32" y="29" smashed="yes" rot="R270">
+<element name="R7" library="adafruit" package="0204V" value="470" x="32" y="29" smashed="yes" rot="R270">
 <attribute name="NAME" x="33.0668" y="28" size="0.8128" layer="25" ratio="12"/>
 <attribute name="VALUE" x="29.6886" y="31.1336" size="1.27" layer="27" ratio="12" rot="R270"/>
 </element>
-<element name="R6" library="adafruit" package="0204V" value="" x="27.5" y="29" smashed="yes" rot="R270">
+<element name="R6" library="adafruit" package="0204V" value="470" x="27.5" y="29" smashed="yes" rot="R270">
 <attribute name="NAME" x="28.5922" y="28" size="0.8128" layer="25" ratio="12"/>
 <attribute name="VALUE" x="25.1886" y="31.1336" size="1.27" layer="27" ratio="12" rot="R270"/>
@@
 <attribute name="VALUE" x="16.849" y="22.595" size="1.27" layer="27" ratio="10" rot="R270"/>
 </element>
-<element name="R5" library="adafruit" package="0204V" value="" x="23" y="29" smashed="yes" rot="R270">
+<element name="R5" library="adafruit" package="0204V" value="470" x="23" y="29" smashed="yes" rot="R270">
 <attribute name="NAME" x="24.0668" y="28" size="0.8128" layer="25" ratio="12"/>
 <attribute name="VALUE" x="20.6886" y="31.1336" size="1.27" layer="27" ratio="12" rot="R270"/>
 </element>
-<element name="R4" library="adafruit" package="0204V" value="" x="18.5" y="29" smashed="yes" rot="R270">
+<element name="R4" library="adafruit" package="0204V" value="470" x="18.5" y="29" smashed="yes" rot="R270">
 <attribute name="NAME" x="19.4906" y="28" size="0.8128" layer="25" ratio="12"/>
 <attribute name="VALUE" x="16.1886" y="31.1336" size="1.27" layer="27" ratio="12" rot="R270"/>
@@
 <attribute name="NAME" x="8.6162" y="9.5" size="0.8128" layer="21" rot="R180"/>
 </element>
-<element name="Q1" library="special" library_urn="urn:adsk.eagle:library:367" package="QS" value="" x="42" y="37" smashed="yes" rot="R90">
+<element name="Q1" library="special" library_urn="urn:adsk.eagle:library:367" package="QS" value="16MHz" x="42" y="37" smashed="yes" rot="R90">
 <attribute name="NAME" x="41" y="30" size="0.8128" layer="25" ratio="10"/>
 <attribute name="VALUE" x="45.937" y="31.92" size="1.27" layer="27" ratio="10" rot="R90"/>
 </element>
-<element name="C2" library="adafruit" package="C025-024X044" value="" x="46.5" y="39.5" smashed="yes" rot="R90">
+<element name="C2" library="adafruit" package="C025-024X044" value="22pF" x="46.5" y="39.5" smashed="yes" rot="R90">
 <attribute name="NAME" x="48.0494" y="37.2902" size="0.8128" layer="25" ratio="10"/>
 <attribute name="VALUE" x="49.167" y="37.722" size="1.27" layer="27" ratio="10" rot="R90"/>
 </element>
-<element name="C3" library="adafruit" package="C025-024X044" value="" x="46.5" y="34" smashed="yes" rot="R270">
+<element name="C3" library="adafruit" package="C025-024X044" value="22pF" x="46.5" y="34" smashed="yes" rot="R270">
 <attribute name="NAME" x="47.9478" y="32.0188" size="0.8128" layer="25" ratio="10"/>
 <attribute name="VALUE" x="43.833" y="35.778" size="1.27" layer="27" ratio="10" rot="R270"/>
 </element>
-<element name="R3" library="adafruit" package="0204V" value="" x="10" y="28" smashed="yes" rot="R270">
+<element name="R3" library="adafruit" package="0204V" value="15k" x="10" y="28" smashed="yes" rot="R270">
 <attribute name="NAME" x="10.7" y="25.5" size="0.8128" layer="25" ratio="12"/>
 <attribute name="VALUE" x="7.6886" y="30.1336" size="1.27" layer="27" ratio="12" rot="R270"/>
 </element>
-<element name="C1" library="adafruit" package="C025-024X044" value="" x="13.5" y="28" smashed="yes" rot="R90">
+<element name="C1" library="adafruit" package="C025-024X044" value=".1uF" x="13.5" y="28" smashed="yes" rot="R90">
 <attribute name="NAME" x="15" y="25.5" size="0.8128" layer="25" ratio="10"/>
 <attribute name="VALUE" x="16.167" y="26.222" size="1.27" layer="27" ratio="10" rot="R90"/>
@@
 <attribute name="VALUE" x="48.12" y="15.92" size="1.27" layer="27" ratio="10" rot="R90"/>
 </element>
-<element name="C4" library="adafruit" package="E2,5-6E" value="" x="48.5" y="26.5" smashed="yes" rot="R90">
+<element name="C4" library="adafruit" package="E2,5-6E" value="4.7uF" x="48.5" y="26.5" smashed="yes" rot="R90">
 <attribute name="NAME" x="51.7512" y="26.8556" size="0.8128" layer="25" ratio="10"/>
 <attribute name="VALUE" x="51.04" y="29.167" size="1.27" layer="27" ratio="10" rot="R90"/>
 </element>
-<element name="C5" library="adafruit" package="E2,5-6E" value="" x="41" y="12" smashed="yes" rot="R180">
+<element name="C5" library="adafruit" package="E2,5-6E" value="0.47uF" x="41" y="12" smashed="yes" rot="R180">
 <attribute name="NAME" x="45.0894" y="14.0066" size="0.8128" layer="25" ratio="10" rot="R180"/>
 <attribute name="VALUE" x="38.333" y="14.54" size="1.27" layer="27" ratio="10" rot="R180"/>
@@
 <attribute name="VALUE" x="8.19" y="43.825" size="1.27" layer="27"/>
 </element>
-<element name="R1" library="adafruit" package="0204V" value="" x="3.5" y="46" smashed="yes" rot="R90">
+<element name="R1" library="adafruit" package="0204V" value="4.7k" x="3.5" y="46" smashed="yes" rot="R90">
 <attribute name="NAME" x="2.82" y="42.9058" size="0.8128" layer="25" ratio="12"/>
 <attribute name="VALUE" x="5.8114" y="43.8664" size="1.27" layer="27" ratio="12" rot="R90"/>
 </element>
-<element name="R2" library="adafruit" package="0204V" value="" x="6" y="46" smashed="yes" rot="R90">
+<element name="R2" library="adafruit" package="0204V" value="4.7k" x="6" y="46" smashed="yes" rot="R90">
 <attribute name="NAME" x="5.4616" y="42.9458" size="0.8128" layer="25" ratio="12"/>
 <attribute name="VALUE" x="8.3114" y="43.8664" size="1.27" layer="27" ratio="12" rot="R90"/>
